File: PCB/HackPad.kicad_sch (KiCad schematic)
At the start: 34 parts, among them SW1 RotaryEncoder_Switch_MP, SW10 SW_Push_45deg, SW11 SW_Push_45deg, SW12 SW_Push_45deg, SW13 SW_Push_45deg, SW14 SW_Push_45deg, SW15 SW_Push_45deg, SW16 SW_Push_45deg, SW17 SW_Push_45deg, SW2 SW_Push_45deg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

Commit message: fixed filee structure
Connections:
- net 3V3: no longer SW1.S2
- net at U1.10 (GPIO4/MISO): now also SW1.S2
Changed lines of the file:
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@@
+	(wire
+		(pts
+			(xy 248.92 105.41) (xy 261.62 105.41)
+		)
+		(stroke
+			(width 0)
+			(type default)
+		)
+	)
 	(wire
 		(pts
@@
 	(wire
 		(pts
+			(xy 261.62 105.41) (xy 261.62 71.12)
+		)
+		(stroke
+			(width 0)
+			(type default)
+		)
+	)
+	(wire
+		(pts
 			(xy 190.5 153.67) (xy 190.5 157.48)
 		)
@@
 	(wire
 		(pts
+			(xy 261.62 71.12) (xy 259.08 71.12)
+		)
+		(stroke
+			(width 0)
+			(type default)
+		)
+	)
+	(wire
+		(pts
 			(xy 175.26 166.37) (xy 195.58 166.37)
 		)
@@
 		(pts
 			(xy 118.11 74.93) (xy 118.11 113.03)
+		)
+		(stroke
+			(width 0)
+			(type default)
+		)
+	)
+	(wire
+		(pts
+			(xy 248.92 105.41) (xy 248.92 104.14)
 		)
 		(stroke
@@
 				(hide yes)
 			)
-		)
-	)
-	(global_label "3V3"
-		(shape input)
-		(at 248.92 104.14 0)
-		(fields_autoplaced yes)
-		(effects
-			(font
-				(size 1.27 1.27)
-			)
-			(justify left)
-		)
-		(property "Intersheetrefs" "${INTERSHEET_REFS}"
-			(at 255.4128 104.14 0)
-			(effects
-				(font
-					(size 1.27 1.27)
-				)
-				(justify left)
-				(hide yes)
-			)

Commit message: Add files via upload
Parts:
- SW11, SW17, SW5: footprint Button_Switch_Keyboard:SW_Cherry_MX_1.00u_PCB -> Button_Switch_Keyboard:SW_Cherry_MX_2.00u_PCB
- SW14: footprint Button_Switch_Keyboard:SW_Cherry_MX_1.75u_PCB -> Button_Switch_Keyboard:SW_Cherry_MX_1.00u_PCB
- SW2, SW3: footprint Button_Switch_Keyboard:SW_Cherry_MX_2.25u_PCB -> Button_Switch_Keyboard:SW_Cherry_MX_1.00u_PCB
Connections:
- net COL1: now also SW12.1, SW13.1, SW9.1
- net COL2: now also SW10.1, SW14.1, SW15.1
- net COL3: now also SW11.1, SW16.1, SW17.1
Changed lines of the file:
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@@
 	)
 	(junction
-		(at 146.05 74.93)
+		(at 170.18 74.93)
 		(diameter 0)
 		(color 0 0 0 0)
 	)
 	(junction
-		(at 170.18 74.93)
+		(at 173.99 45.72)
 		(diameter 0)
 		(color 0 0 0 0)
 	)
 	(junction
-		(at 173.99 45.72)
+		(at 146.05 74.93)
 		(diameter 0)
 		(color 0 0 0 0)
@@
 	(wire
 		(pts
+			(xy 146.05 74.93) (xy 146.05 33.02)
+		)
+		(stroke
+			(width 0)
+			(type default)
+		)
+	)
+	(wire
+		(pts
 			(xy 151.13 125.73) (xy 175.26 125.73)
 		)
@@
 	(wire
 		(pts
-			(xy 190.5 34.29) (xy 190.5 74.93)
+			(xy 146.05 33.02) (xy 144.78 33.02)
 		)
 		(stroke
@@
 	(wire
 		(pts
-			(xy 259.08 85.09) (xy 259.08 78.74)
+			(xy 170.18 33.02) (xy 170.18 74.93)
 		)
 		(stroke
@@
 	(wire
 		(pts
-			(xy 146.05 113.03) (xy 146.05 153.67)
+			(xy 259.08 85.09) (xy 259.08 78.74)
 		)
 		(stroke
@@
 	(wire
 		(pts
-			(xy 170.18 34.29) (xy 170.18 74.93)
+			(xy 146.05 113.03) (xy 146.05 153.67)
 		)
 		(stroke
@@
 	(wire
 		(pts
-			(xy 195.58 166.37) (xy 212.09 166.37)
+			(xy 170.18 33.02) (xy 168.91 33.02)
 		)
 		(stroke
@@
 	(wire
 		(pts
-			(xy 149.86 45.72) (xy 173.99 45.72)
+			(xy 195.58 166.37) (xy 212.09 166.37)
 		)
 		(stroke
@@
 	(wire
 		(pts
-			(xy 195.58 125.73) (xy 210.82 125.73)
+			(xy 149.86 45.72) (xy 173.99 45.72)
 		)
 		(stroke
@@
 	(wire
 		(pts
-			(xy 233.68 85.09) (xy 259.08 85.09)
+			(xy 195.58 125.73) (xy 210.82 125.73)
 		)
 		(stroke
@@
 	(wire
 		(pts
-			(xy 212.09 166.37) (xy 212.09 167.64)
+			(xy 233.68 85.09) (xy 259.08 85.09)
 		)
 		(stroke
@@
 	(wire
 		(pts
-			(xy 146.05 34.29) (xy 146.05 74.93)
+			(xy 212.09 166.37) (xy 212.09 167.64)
 		)
 		(stroke
@@
 	(wire
 		(pts
+			(xy 190.5 33.02) (xy 189.23 33.02)
+		)
+		(stroke
+			(width 0)
+			(type default)
+		)
+	)
+	(wire
+		(pts
 			(xy 175.26 166.37) (xy 195.58 166.37)
 		)
@@
 	(wire
 		(pts
+			(xy 190.5 33.02) (xy 190.5 74.93)
+		)
+		(stroke
+			(width 0)
+			(type default)
+		)
+	)
+	(wire
+		(pts
 			(xy 195.58 87.63) (xy 212.09 87.63)
 		)
@@
 			)
 		)
-		(property "Footprint" "Button_Switch_Keyboard:SW_Cherry_MX_1.75u_PCB"
+		(property "Footprint" "Button_Switch_Keyboard:SW_Cherry_MX_1.00u_PCB"
 			(at 172.72 77.47 0)
 			(effects
@@
 			)
 		)
-		(property "Footprint" "Button_Switch_Keyboard:SW_Cherry_MX_2.25u_PCB"
+		(property "Footprint" "Button_Switch_Keyboard:SW_Cherry_MX_1.00u_PCB"
 			(at 147.32 35.56 0)
 			(effects
@@
 			)
 		)
-		(property "Footprint" "Button_Switch_Keyboard:SW_Cherry_MX_2.25u_PCB"
+		(property "Footprint" "Button_Switch_Keyboard:SW_Cherry_MX_1.00u_PCB"
 			(at 120.65 35.56 0)
 			(effects
@@
 			)
 		)
-		(property "Footprint" "Button_Switch_Keyboard:SW_Cherry_MX_1.00u_PCB"
+		(property "Footprint" "Button_Switch_Keyboard:SW_Cherry_MX_2.00u_PCB"
 			(at 193.04 77.47 0)
 			(effects
@@
 			)
 		)
-		(property "Footprint" "Button_Switch_Keyboard:SW_Cherry_MX_1.00u_PCB"
+		(property "Footprint" "Button_Switch_Keyboard:SW_Cherry_MX_2.00u_PCB"
 			(at 191.77 35.56 0)
 			(effects
@@
 			)
 		)
-		(property "Footprint" "Button_Switch_Keyboard:SW_Cherry_MX_1.00u_PCB"
+		(property "Footprint" "Button_Switch_Keyboard:SW_Cherry_MX_2.00u_PCB"
 			(at 193.04 156.21 0)
 			(effects
